File: Audio/PCB Design/SplitAudio/SplitAudio.sch (KiCad schematic (older format))
At the start: 6 parts, among them J1 AudioJack3, J2 AudioJack3, SW1 SW_Push, SW2 SW_Push, U1 DFPLAYER_MINI

Commit message: Audio board completed
Parts:
- removed J1, J2: AudioJack3, Connector_Audio:Jack_3.5mm_PJ311_Horizontal, symbol Connector:AudioJack3
- added J1, J2: 35RAPC4BH3, AudioJack:SWITCHCRAFT_35RAPC4BH3, symbol 35RAPC4BH3:35RAPC4BH3
Connections:
- net at U1.4 (DAC_R): now also J1.2
- net at U1.7 (GND): now also J1.1, J2.1
- net at U1.5 (DAC_L): now also J2.5
- no-connect marks 12 -> 16
Changed lines of the file:
@@
-$EndComp
-$Comp
-L Connector:AudioJack3 J1
-U 1 1 5C6D2B8D
-P 4550 2750
-F 0 "J1" H 4530 3075 50  0000 C CNN
-F 1 "AudioJack3" H 4530 2984 50  0000 C CNN
-F 2 "Connector_Audio:Jack_3.5mm_PJ311_Horizontal" H 4550 2750 50  0001 C CNN
-F 3 "~" H 4550 2750 50  0001 C CNN
-	1    4550 2750
-	1    0    0    -1
-$EndComp
-$Comp
-L Connector:AudioJack3 J2
-U 1 1 5C6D2BC9
-P 4550 3900
-F 0 "J2" H 4530 4225 50  0000 C CNN
-F 1 "AudioJack3" H 4530 4134 50  0000 C CNN
-F 2 "Connector_Audio:Jack_3.5mm_PJ311_Horizontal" H 4550 3900 50  0001 C CNN
-F 3 "~" H 4550 3900 50  0001 C CNN
-	1    4550 3900
-	1    0    0    -1
 $EndComp
 $Comp
@@
 	6000 3200 5200 3200
 Wire Wire Line
-	5200 3200 5200 4000
-Wire Wire Line
-	5200 4000 4750 4000
-NoConn ~ 4750 2850
+	5200 4200 4750 4200
 NoConn ~ 4750 3900
 $Comp
@@
 Wire Wire Line
 	7150 2150 6000 2150
+$Comp
+L 35RAPC4BH3:35RAPC4BH3 J1
+U 1 1 5C6D5449
+P 4250 2850
+F 0 "J1" H 4355 3317 50  0000 C CNN
+F 1 "35RAPC4BH3" H 4355 3226 50  0000 C CNN
+F 2 "AudioJack:SWITCHCRAFT_35RAPC4BH3" H 4250 2850 50  0001 L BNN
+F 3 "35RAPC4BH3" H 4250 2850 50  0001 L BNN
+F 4 "Unavailable" H 4250 2850 50  0001 L BNN "Field4"
+F 5 "Switchcraft Inc." H 4250 2850 50  0001 L BNN "Field5"
+F 6 "None" H 4250 2850 50  0001 L BNN "Field6"
+F 7 "3.5mm Threaded Right Angle Stereo Jack" H 4250 2850 50  0001 L BNN "Field7"
+F 8 "None" H 4250 2850 50  0001 L BNN "Field8"
+	1    4250 2850
+	1    0    0    -1
+$EndComp
+$Comp
+L 35RAPC4BH3:35RAPC4BH3 J2
+U 1 1 5C6D5508
+P 4250 4000
+F 0 "J2" H 4355 4467 50  0000 C CNN
+F 1 "35RAPC4BH3" H 4355 4376 50  0000 C CNN
+F 2 "AudioJack:SWITCHCRAFT_35RAPC4BH3" H 4250 4000 50  0001 L BNN
+F 3 "35RAPC4BH3" H 4250 4000 50  0001 L BNN
+F 4 "Unavailable" H 4250 4000 50  0001 L BNN "Field4"
+F 5 "Switchcraft Inc." H 4250 4000 50  0001 L BNN "Field5"
+F 6 "None" H 4250 4000 50  0001 L BNN "Field6"
+F 7 "3.5mm Threaded Right Angle Stereo Jack" H 4250 4000 50  0001 L BNN "Field7"
+F 8 "None" H 4250 4000 50  0001 L BNN "Field8"
+	1    4250 4000
+	1    0    0    -1
+$EndComp
+Wire Wire Line
+	5200 3200 5200 4200
+NoConn ~ 4750 2850
+NoConn ~ 4750 2950
+NoConn ~ 4750 3050
+NoConn ~ 4750 4000
+NoConn ~ 4750 4100
 $EndSCHEMATC
